Commit message: update urdf

File: src/inspire_franka_description/urdf/inspire_franka.urdf.xacro (robot description, xacro)
@@ -7,7 +7,6 @@
   workspace, which is exactly how the real setup is wired (one FCI connection,
   one USB-RS485 adapter, no mechanical coupling).
-  `hand_mount:=flange` bolts the hand to the arm's flange instead. The
-  kinematics for that are here and correct in orientation, but the OFFSET IS A
-  PLACEHOLDER - see hand_flange_xyz below.
+  `hand_mount:=flange` bolts the hand to the arm's flange instead, using the
+  same fr3_link8-to-palm transform as forgeUltra's franka-chi asset.
       xacro inspire_franka.urdf.xacro                          # arm + bench hand
       xacro inspire_franka.urdf.xacro hand:=false              # bare arm
@@ -112,14 +111,13 @@
     <xacro:property name="hand_bench_rpy" value="0 0 0"/>
     <!--
-      PLACEHOLDER. The rotation is right - the fingers point away from the flange
-      along the arm's approach axis, which is what an identity rotation gives -
-      but 10 mm is a guess at the adapter plate's thickness, and there is no
-      measured clocking angle about z.
-      To fix: measure the adapter, set hand_flange_xyz to its true thickness and
-      hand_flange_rpy's yaw to how the hand is clocked on it. Until then, treat
-      any flange-mounted fingertip pose as approximate.
+      Match forgeUltra's franka-chi asset, which welds fr3_link8 directly to
+      palm at zero translation with q_wxyz=(0.5, -0.5, -0.5, 0.5).
+      This description has an intermediate hand_mount frame. Its fixed
+      base_joint contributes rpy=(-pi/2, 0, pi), so applying a -pi/2 yaw here
+      gives the same composed fr3_link8-to-hand_base_link (palm) transform.
+      Keep these values synchronized with inspire_hand_on_flange.xml.
     -->
-    <xacro:property name="hand_flange_xyz" value="0 0 0.010"/>
-    <xacro:property name="hand_flange_rpy" value="0 0 0"/>
+    <xacro:property name="hand_flange_xyz" value="0 0 0"/>
+    <xacro:property name="hand_flange_rpy" value="0 0 -1.5707963267948966"/>
     <xacro:property name="hand_parent_resolved"
       value="${arm_link_prefix + 'link8' if mount == 'flange'

Commit message: Checkpoint unified simulation and trajectory replay

File: src/inspire_franka_description/urdf/inspire_franka.urdf.xacro (robot description, xacro)
@@ -2,15 +2,10 @@
 <!--
   The Franka FR3 and the Inspire RH56 hand in one description.
-  By default they are two separate objects sharing a world: the arm at the
-  origin, the hand standing on the bench beside it. That is the "bench hand"
-  arrangement - the two are independent assets that happen to be in the same
-  workspace, which is exactly how the real setup is wired (one FCI connection,
-  one USB-RS485 adapter, no mechanical coupling).
-  `hand_mount:=flange` bolts the hand to the arm's flange instead, using the
-  same fr3_link8-to-palm transform as forgeUltra's franka-chi asset.
-      xacro inspire_franka.urdf.xacro                          # arm + bench hand
+  When both assets are enabled, the hand is always bolted to the arm's flange
+  using the same fr3_link8-to-palm transform as forgeUltra's franka-chi asset.
+  With only one asset enabled, that asset is described on its own.
+      xacro inspire_franka.urdf.xacro                          # arm + flange hand
       xacro inspire_franka.urdf.xacro hand:=false              # bare arm
       xacro inspire_franka.urdf.xacro arm:=false               # hand only
-      xacro inspire_franka.urdf.xacro hand_mount:=flange       # hand on the flange
   ros2_control here is SIMULATION ONLY (`mujoco` or `mock`). The real arm goes
   through upstream franka_bringup and the real hand through inspire_hand_driver;
@@ -30,11 +25,4 @@
   <xacro:arg name="hand_side" default="right"/>
   <xacro:arg name="hand_prefix" default=""/>
-  <!-- 'bench'  - the hand stands on the table beside the arm, unattached.
-       'flange' - the hand is bolted to the arm's flange (fr3_link8).
-       'custom' - use hand_xyz/hand_rpy verbatim, against hand_parent. -->
-  <xacro:arg name="hand_mount" default="bench"/>
-  <xacro:arg name="hand_parent" default="world"/>
-  <xacro:arg name="hand_xyz" default="0 0 0"/>
-  <xacro:arg name="hand_rpy" default="0 0 0"/>
   <!-- ros2_control, for simulation. -->
   <xacro:arg name="ros2_control" default="false"/>
@@ -55,5 +43,4 @@
   <xacro:property name="with_arm" value="$(arg arm)"/>
   <xacro:property name="with_hand" value="$(arg hand)"/>
-  <xacro:property name="mount" value="$(arg hand_mount)"/>
   <!--
     Guards. A silent empty or half-built URDF is a miserable thing to debug, so
@@ -69,10 +56,4 @@
   <xacro:unless value="${with_arm or with_hand}">
     <link name="${dict()['inspire_franka: arm and hand are both false, so there is nothing to describe. Set arm:=true or hand:=true.']}"/>
-  </xacro:unless>
-  <xacro:if value="${mount == 'flange' and not with_arm}">
-    <link name="${dict()['inspire_franka: hand_mount:=flange needs an arm to bolt the hand to, but arm:=false.']}"/>
-  </xacro:if>
-  <xacro:unless value="${mount in ('bench', 'flange', 'custom')}">
-    <link name="${dict()['inspire_franka: hand_mount must be bench, flange or custom.']}"/>
   </xacro:unless>
   <!-- franka_arm creates its own `connected_to` link, so `world` comes from the
@@ -101,34 +82,17 @@
       value="${('$(arg arm_prefix)' + '_' if '$(arg arm_prefix)' else '') + '$(arg robot_type)' + '_'}"/>
     <!--
-      Bench pose: 0.45 m forward and 0.35 m to the arm's right, standing on the
-      table. 0.57 m from the base, comfortably inside the FR3's reach, so the
-      arm can be driven to touch the hand.
-      Orientation: hand_mount's +z is the direction the fingers point (the
-      vendored model's base_joint rotates hand_base_link's -y onto +z), so an
-      identity rotation stands the hand upright on the bench.
-    -->
-    <xacro:property name="hand_bench_xyz" value="0.45 -0.35 0.0"/>
-    <xacro:property name="hand_bench_rpy" value="0 0 0"/>
-    <!--
-      Match forgeUltra's franka-chi asset, which welds fr3_link8 directly to
-      palm at zero translation with q_wxyz=(0.5, -0.5, -0.5, 0.5).
-      This description has an intermediate hand_mount frame. Its fixed
-      base_joint contributes rpy=(-pi/2, 0, pi), so applying a -pi/2 yaw here
-      gives the same composed fr3_link8-to-hand_base_link (palm) transform.
+      Mount hand_mount directly on fr3_link8 with a 180-degree clocking angle. The
+      hand's fixed base_joint still defines the model-internal
+      hand_mount-to-hand_base_link orientation.
       Keep these values synchronized with inspire_hand_on_flange.xml.
     -->
     <xacro:property name="hand_flange_xyz" value="0 0 0"/>
-    <xacro:property name="hand_flange_rpy" value="0 0 -1.5707963267948966"/>
+    <xacro:property name="hand_flange_rpy" value="0 0 3.141592653589793"/>
     <xacro:property name="hand_parent_resolved"
-      value="${arm_link_prefix + 'link8' if mount == 'flange'
-              else '$(arg hand_parent)'}"/>
+      value="${arm_link_prefix + 'link8' if with_arm else 'world'}"/>
     <xacro:property name="hand_xyz_resolved"
-      value="${hand_flange_xyz if mount == 'flange'
-              else hand_bench_xyz if mount == 'bench'
-              else '$(arg hand_xyz)'}"/>
+      value="${hand_flange_xyz if with_arm else '0 0 0.2'}"/>
     <xacro:property name="hand_rpy_resolved"
-      value="${hand_flange_rpy if mount == 'flange'
-              else hand_bench_rpy if mount == 'bench'
-              else '$(arg hand_rpy)'}"/>
+      value="${hand_flange_rpy if with_arm else '0 0 0'}"/>
     <xacro:inspire_hand
       side="$(arg hand_side)"

Commit message: fix arm_hand asset mismatch

File: src/inspire_franka_description/urdf/inspire_franka.urdf.xacro (robot description, xacro)
@@ -4,9 +4,9 @@
   By default they are two separate objects sharing a world: the arm at the
   origin, the hand standing on the bench beside it. That is the "bench hand"
-  arrangement - the two are independent assets that happen to be in the same
-  workspace, which is exactly how the real setup is wired (one FCI connection,
-  one USB-RS485 adapter, no mechanical coupling).
-  `hand_mount:=flange` bolts the hand to the arm's flange instead, using the
-  same fr3_link8-to-palm transform as forgeUltra's franka-chi asset.
+  arrangement, useful when bringing up either device independently. The real
+  installation uses the flange mount below while retaining separate FCI and
+  USB-RS485 control connections.
+  `hand_mount:=flange` bolts the hand to the arm's flange instead, matching the
+  90-degree clocking of the hand from the legacy physical installation.
       xacro inspire_franka.urdf.xacro                          # arm + bench hand
       xacro inspire_franka.urdf.xacro hand:=false              # bare arm
@@ -111,13 +111,13 @@
     <xacro:property name="hand_bench_rpy" value="0 0 0"/>
     <!--
-      Match forgeUltra's franka-chi asset, which welds fr3_link8 directly to
-      palm at zero translation with q_wxyz=(0.5, -0.5, -0.5, 0.5).
       This description has an intermediate hand_mount frame. Its fixed
-      base_joint contributes rpy=(-pi/2, 0, pi), so applying a -pi/2 yaw here
-      gives the same composed fr3_link8-to-hand_base_link (palm) transform.
+      base_joint contributes rpy=(-pi/2, 0, pi). The current physical hand is
+      flipped from the zero-yaw pose and is 90 degrees from the legacy
+      installation after angle wrapping, so the flange adapter uses a pi yaw.
+      The 10 mm z offset is the thickness of the black physical adapter flange.
       Keep these values synchronized with inspire_hand_on_flange.xml.
     -->
-    <xacro:property name="hand_flange_xyz" value="0 0 0"/>
-    <xacro:property name="hand_flange_rpy" value="0 0 -1.5707963267948966"/>
+    <xacro:property name="hand_flange_xyz" value="0 0 0.010"/>
+    <xacro:property name="hand_flange_rpy" value="0 0 3.141592653589793"/>
     <xacro:property name="hand_parent_resolved"
       value="${arm_link_prefix + 'link8' if mount == 'flange'
@@ -131,4 +131,24 @@
               else hand_bench_rpy if mount == 'bench'
               else '$(arg hand_rpy)'}"/>
+    <!-- The mesh is centred on a frame 5 mm above link8, so its faces span
+         z=0..10 mm and meet both the wrist and the translated hand palm. -->
+    <xacro:if value="${mount == 'flange'}">
+      <link name="$(arg hand_prefix)hand_adapter_flange">
+        <visual>
+          <origin xyz="0 0 0" rpy="0 0 0"/>
+          <geometry>
+            <mesh filename="package://inspire_franka_description/meshes/adapter_flange.stl"/>
+          </geometry>
+          <material name="hand_adapter_flange_black">
+            <color rgba="0.025 0.025 0.025 1"/>
+          </material>
+        </visual>
+      </link>
+      <joint name="$(arg hand_prefix)hand_adapter_flange_joint" type="fixed">
+        <origin xyz="0 0 0.005" rpy="0 0 0"/>
+        <parent link="${arm_link_prefix}link8"/>
+        <child link="$(arg hand_prefix)hand_adapter_flange"/>
+      </joint>
+    </xacro:if>
     <xacro:inspire_hand
       side="$(arg hand_side)"
